File: FC002B (Production PCB)/KiCAD/FC003.sch (KiCad schematic (older format))
At the start: 50 parts, among them IC1 MSP430G2202, IC10 SC52-11, IC11 SC52-11, IC12 SC52-11, IC2 4017, IC3 74HC4060, IC4 ULN2803A, IC5 SC52-11, IC6 SC52-11, IC7 SC52-11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

Commit message: F003 Schematic 20131202_1
Parts:
- added J?: HF SRC, SIL-2, symbol CONN_2
- IC2: footprint (none) -> DIP-16__300_ELL
- IC4: footprint ~ -> DIP-18__300_ELL
- J10, J11, J12, J13, J14, J7, J8, J9: footprint (none) -> SIL-2
Connections:
- net at IC1.19 (P2.6/XIN): now also J5.2 (PM), J?.2 (PM); no longer IC3.9 (CTC)
- net at IC1.3 (P1.1): now also J5.1 (P1)
- new net: IC3.9 (CTC), J?.1 (P1)
Other:
- moved on the sheet: J2, J5

Commit message: FC003 - Schematic 20131203_2
Parts:
- added D10, D9: 1N4148, D3, symbol DIODE
- added R4: 1M, R4, symbol R
- added R5: 10K, R4, symbol R
- D1, D2, D3, D4, D5, D6, D7, D8: value DIODE -> 1N4148; footprint (none) -> D3
- gave numbers to parts that had none: 1
Connections:
- net GND: now also D10.1 (A), R4.2
- net VCC: now also D9.2 (K)
- net at IC1.2 (P1.0), IC1.6 (P1.4): now also D10.2 (K), D9.1 (A), R5.2; no longer J2.1 (P1)
- new net: J2.1 (P1), R4.1, R5.1
Changed lines of the file:
@@
 LIBS:contrib
 LIBS:valves
-LIBS:FC003-cache
 EELAYER 27 0
 EELAYER END
@@
 	3700 4725 4425 4725
 Wire Wire Line
-	1800 4625 2300 4625
-Wire Wire Line
-	1800 2525 1800 4625
+	2100 4625 2300 4625
+Wire Wire Line
+	2100 2525 2100 4625
 Wire Wire Line
 	4375 2150 4375 2200
@@
 Wire Wire Line
 	4300 4575 4300 4725
-Wire Wire Line
-	1250 4425 2300 4425
 Wire Wire Line
 	1250 5150 1250 5300
@@
 8x Kingbright SC52-11
 $Comp
-L GND #PWR8
+L GND #PWR7
 U 1 1 513EAE8F
 P 3825 1400
-F 0 "#PWR8" H 3825 1400 30  0001 C CNN
+F 0 "#PWR7" H 3825 1400 30  0001 C CNN
 F 1 "GND" H 3825 1330 30  0001 C CNN
 F 2 "" H 3825 1400 60  0001 C CNN
@@
 $EndComp
 $Comp
-L GND #PWR15
+L GND #PWR2
 U 1 1 513AC4CA
 P 1250 5300
-F 0 "#PWR15" H 1250 5300 30  0001 C CNN
+F 0 "#PWR2" H 1250 5300 30  0001 C CNN
 F 1 "GND" H 1250 5230 30  0001 C CNN
 F 2 "" H 1250 5300 60  0001 C CNN
@@
 $EndComp
 $Comp
-L VCC #PWR16
+L VCC #PWR14
 U 1 1 512E956E
 P 8000 1325
-F 0 "#PWR16" H 8000 1425 30  0001 C CNN
+F 0 "#PWR14" H 8000 1425 30  0001 C CNN
 F 1 "VCC" H 8000 1425 30  0000 C CNN
 F 2 "" H 8000 1325 60  0001 C CNN
@@
 $EndComp
 $Comp
-L GND #PWR17
+L GND #PWR15
 U 1 1 512E9564
 P 8000 1975
-F 0 "#PWR17" H 8000 1975 30  0001 C CNN
+F 0 "#PWR15" H 8000 1975 30  0001 C CNN
 F 1 "GND" H 8000 1905 30  0001 C CNN
 F 2 "" H 8000 1975 60  0001 C CNN
@@
 $EndComp
 $Comp
-L GND #PWR3
+L GND #PWR1
 U 1 1 512D1F12
 P 1250 4725
-F 0 "#PWR3" H 1250 4725 30  0001 C CNN
+F 0 "#PWR1" H 1250 4725 30  0001 C CNN
 F 1 "GND" H 1250 4725 60  0001 C CNN
 F 2 "" H 1250 4725 60  0001 C CNN
@@
 $EndComp
 $Comp
-L GND #PWR13
+L GND #PWR12
 U 1 1 512D1EB3
 P 4425 4950
-F 0 "#PWR13" H 4425 4950 30  0001 C CNN
+F 0 "#PWR12" H 4425 4950 30  0001 C CNN
 F 1 "GND" H 4425 4950 60  0001 C CNN
 F 2 "" H 4425 4950 60  0001 C CNN
@@
 $EndComp
 $Comp
-L VCC #PWR11
+L VCC #PWR10
 U 1 1 512C3C5B
 P 4375 675
-F 0 "#PWR11" H 4375 775 30  0001 C CNN
+F 0 "#PWR10" H 4375 775 30  0001 C CNN
 F 1 "VCC" H 4375 675 60  0001 C CNN
 F 2 "" H 4375 675 60  0001 C CNN
@@
 $EndComp
 $Comp
-L GND #PWR12
+L GND #PWR11
 U 1 1 512C3C4C
 P 4375 2200
-F 0 "#PWR12" H 4375 2200 30  0001 C CNN
+F 0 "#PWR11" H 4375 2200 30  0001 C CNN
 F 1 "GND" H 4375 2200 60  0001 C CNN
 F 2 "" H 4375 2200 60  0001 C CNN
@@
 $EndComp
 $Comp
-L GND #PWR7
+L GND #PWR6
 U 1 1 5127F6B0
 P 3425 2425
-F 0 "#PWR7" H 3425 2425 30  0001 C CNN
+F 0 "#PWR6" H 3425 2425 30  0001 C CNN
 F 1 "GND" H 3425 2355 30  0001 C CNN
 F 2 "" H 3425 2425 60  0001 C CNN
@@
 $EndComp
 $Comp
-L VCC #PWR10
+L VCC #PWR9
 U 1 1 51268761
 P 4300 4150
-F 0 "#PWR10" H 4300 4250 30  0001 C CNN
+F 0 "#PWR9" H 4300 4250 30  0001 C CNN
 F 1 "VCC" H 4300 4250 30  0000 C CNN
 F 2 "" H 4300 4150 60  0001 C CNN
@@
 $EndComp
 $Comp
-L VCC #PWR5
+L VCC #PWR4
 U 1 1 51228951
 P 2300 4150
-F 0 "#PWR5" H 2300 4250 30  0001 C CNN
+F 0 "#PWR4" H 2300 4250 30  0001 C CNN
 F 1 "VCC" H 2300 4250 30  0000 C CNN
 F 2 "" H 2300 4150 60  0001 C CNN
@@
 $EndComp
 $Comp
-L GND #PWR9
+L GND #PWR8
 U 1 1 51228936
 P 4100 5275
-F 0 "#PWR9" H 4100 5275 30  0001 C CNN
+F 0 "#PWR8" H 4100 5275 30  0001 C CNN
 F 1 "GND" H 4100 5205 30  0001 C CNN
 F 2 "" H 4100 5275 60  0001 C CNN
@@
 $EndComp
 $Comp
-L GND #PWR14
+L GND #PWR13
 U 1 1 528EEC3C
 P 4500 3600
-F 0 "#PWR14" H 4500 3600 30  0001 C CNN
+F 0 "#PWR13" H 4500 3600 30  0001 C CNN
 F 1 "GND" H 4500 3530 30  0001 C CNN
 F 2 "" H 4500 3600 60  0000 C CNN
@@
 P 9075 4700
 F 0 "D1" H 9175 4725 40  0000 C CNN
-F 1 "DIODE" H 8925 4725 40  0000 C CNN
-F 2 "" H 9075 4700 60  0000 C CNN
+F 1 "1N4148" H 8925 4725 40  0000 C CNN
+F 2 "D3" H 9075 4700 60  0001 C CNN
 F 3 "" H 9075 4700 60  0000 C CNN
 	1    9075 4700
@@
 P 9225 4700
 F 0 "D2" H 9325 4725 40  0000 C CNN
-F 1 "DIODE" H 9075 4725 40  0000 C CNN
-F 2 "" H 9225 4700 60  0000 C CNN
+F 1 "1N4148" H 9075 4725 40  0000 C CNN
+F 2 "D3" H 9225 4700 60  0001 C CNN
 F 3 "" H 9225 4700 60  0000 C CNN
 	1    9225 4700
@@
 P 9375 4700
 F 0 "D3" H 9475 4725 40  0000 C CNN
-F 1 "DIODE" H 9225 4725 40  0000 C CNN
-F 2 "" H 9375 4700 60  0000 C CNN
+F 1 "1N4148" H 9225 4725 40  0000 C CNN
+F 2 "D3" H 9375 4700 60  0001 C CNN
 F 3 "" H 9375 4700 60  0000 C CNN
 	1    9375 4700
@@
 P 9525 4700
 F 0 "D4" H 9625 4725 40  0000 C CNN
-F 1 "DIODE" H 9375 4725 40  0000 C CNN
-F 2 "" H 9525 4700 60  0000 C CNN
+F 1 "1N4148" H 9375 4725 40  0000 C CNN
+F 2 "D3" H 9525 4700 60  0001 C CNN
 F 3 "" H 9525 4700 60  0000 C CNN
 	1    9525 4700
@@
 P 9675 4700
 F 0 "D5" H 9775 4725 40  0000 C CNN
-F 1 "DIODE" H 9525 4725 40  0000 C CNN
-F 2 "" H 9675 4700 60  0000 C CNN
+F 1 "1N4148" H 9525 4725 40  0000 C CNN
+F 2 "D3" H 9675 4700 60  0001 C CNN
 F 3 "" H 9675 4700 60  0000 C CNN
 	1    9675 4700
@@
 P 9825 4700
 F 0 "D6" H 9925 4725 40  0000 C CNN
-F 1 "DIODE" H 9675 4725 40  0000 C CNN
-F 2 "" H 9825 4700 60  0000 C CNN
+F 1 "1N4148" H 9675 4725 40  0000 C CNN
+F 2 "D3" H 9825 4700 60  0001 C CNN
 F 3 "" H 9825 4700 60  0000 C CNN
 	1    9825 4700
@@
 P 9975 4700
 F 0 "D7" H 10075 4725 40  0000 C CNN
-F 1 "DIODE" H 9825 4725 40  0000 C CNN
-F 2 "" H 9975 4700 60  0000 C CNN
+F 1 "1N4148" H 9825 4725 40  0000 C CNN
+F 2 "D3" H 9975 4700 60  0001 C CNN
 F 3 "" H 9975 4700 60  0000 C CNN
 	1    9975 4700
@@
 P 10125 4700
 F 0 "D8" H 10225 4725 40  0000 C CNN
-F 1 "DIODE" H 9975 4725 40  0000 C CNN
-F 2 "" H 10125 4700 60  0000 C CNN
+F 1 "1N4148" H 9975 4725 40  0000 C CNN
+F 2 "D3" H 10125 4700 60  0001 C CNN
 F 3 "" H 10125 4700 60  0000 C CNN
 	1    10125 4700
@@
 Connection ~ 2200 4425
 $Comp
-L GND #PWR6
+L GND #PWR5
 U 1 1 528FE74A
 P 2925 3075
-F 0 "#PWR6" H 2925 3075 30  0001 C CNN
+F 0 "#PWR5" H 2925 3075 30  0001 C CNN
 F 1 "GND" H 2925 3005 30  0001 C CNN
 F 2 "" H 2925 3075 60  0000 C CNN
@@
 	2150 2675 2150 4725
 Wire Wire Line
-	3000 2975 2075 2975
-Wire Wire Line
-	2075 2975 2075 4925
-Wire Wire Line
-	2075 4925 2300 4925
+	3000 2975 2050 2975
+Wire Wire Line
+	2050 2975 2050 4925
+Wire Wire Line
+	2050 4925 2300 4925
 Wire Wire Line
 	4875 1900 4875 2525
 Wire Wire Line
-	4875 2525 1800 2525
+	4875 2525 2100 2525
 Wire Wire Line
 	3700 4825 4025 4825
@@
 	1250 4625 1250 4725
 Wire Wire Line
-	2300 4525 1350 4525
-Wire Wire Line
-	1350 4525 1350 4950
-Wire Wire Line
-	1350 4950 1250 4950
-$Comp
-L CONN_2 J?
+	2300 4525 1950 4525
+Wire Wire Line
+	1950 4525 1950 4950
+Wire Wire Line
+	1950 4950 1250 4950
+$Comp
+L CONN_2 J6
 U 1 1 529D6481
 P 900 3825
-F 0 "J?" V 850 3825 40  0000 C CNN
+F 0 "J6" V 850 3825 40  0000 C CNN
 F 1 "HF SRC" V 950 3825 40  0000 C CNN
 F 2 "SIL-2" H 900 3825 60  0001 C CNN
@@
 	1250 1000 1250 3725
 Wire Wire Line
-	1250 5050 1400 5050
-Wire Wire Line
-	1400 5050 1400 3925
-Connection ~ 1400 3925
+	1250 5050 2000 5050
+Wire Wire Line
+	2000 5050 2000 3925
+Connection ~ 2000 3925
+$Comp
+L R R4
+U 1 1 529D9765
+P 1375 4625
+F 0 "R4" H 1375 4550 40  0000 C CNN
+F 1 "1M" H 1375 4700 40  0000 C CNN
+F 2 "R4" H 1375 4625 60  0001 C CNN
+F 3 "~" H 1375 4625 60  0000 C CNN
+	1    1375 4625
+	0    1    1    0
+$EndComp
+Wire Wire Line
+	1375 4825 1375 5150
+Wire Wire Line
+	1250 5150 1850 5150
+Wire Wire Line
+	1825 4425 2300 4425
+Wire Wire Line
+	1250 4425 1425 4425
+$Comp
+L R R5
+U 1 1 529D9B2F
+P 1625 4425
+F 0 "R5" H 1625 4350 40  0000 C CNN
+F 1 "10K" H 1625 4500 40  0000 C CNN
+F 2 "R4" H 1625 4425 60  0001 C CNN
+F 3 "~" H 1625 4425 60  0000 C CNN
+	1    1625 4425
+	1    0    0    -1
+$EndComp
+Connection ~ 1375 4425
+$Comp
+L DIODE D9
+U 1 1 529D9D87
+P 1850 4175
+F 0 "D9" H 1850 4275 40  0000 C CNN
+F 1 "1N4148" H 1850 4075 40  0000 C CNN
+F 2 "D3" H 1850 4175 60  0001 C CNN
+F 3 "" H 1850 4175 60  0000 C CNN
+	1    1850 4175
+	0    -1   -1   0
+$EndComp
+$Comp
+L DIODE D10
+U 1 1 529D9D99
+P 1850 4675
+F 0 "D10" H 1850 4775 40  0000 C CNN
+F 1 "1N4148" H 1850 4575 40  0000 C CNN
+F 2 "D3" H 1850 4675 60  0001 C CNN
+F 3 "" H 1850 4675 60  0000 C CNN
+	1    1850 4675
+	0    -1   -1   0
+$EndComp
+Wire Wire Line
+	1850 4375 1850 4475
+Connection ~ 1850 4425
+Wire Wire Line
+	1850 5150 1850 4875
+Connection ~ 1375 5150
+$Comp
+L VCC #PWR3
+U 1 1 529DA114
+P 1850 3850
+F 0 "#PWR3" H 1850 3950 30  0001 C CNN
+F 1 "VCC" H 1850 3950 30  0000 C CNN
+F 2 "" H 1850 3850 60  0000 C CNN
+F 3 "" H 1850 3850 60  0000 C CNN
+	1    1850 3850
+	1    0    0    -1
+$EndComp
+Wire Wire Line
+	1850 3975 1850 3850
 $EndSCHEMATC
